File: kicad/luz/luz.kicad_sch (KiCad schematic)
At the start: 58 parts, among them J1 Barrel_Jack, J2 Screw_Terminal_01x04, Q1 AO3400A, Q4 AO3400A, U1 U261-241N-4BS2SS, U2 CYPD3177-24LQXQ_C2959321, U4 TPS54302, U5 ESP32-WROOM-32D

Commit message: Naming schematic values
Parts:
- L1: value SWPA4030S470MT -> 47uH
Changed lines of the file:
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@@
       (effects (font (size 1.27 1.27)))
     )
-    (property "Value" "SWPA4030S470MT" (at 85.725 152.4 0)
+    (property "Value" "47uH" (at 85.725 152.4 0)
       (effects (font (size 1.27 1.27)))
     )

Commit message: Sent 0.0.2a for production
Parts:
- J2: now not fitted
- JP1, JP2, U5: now left out of the parts list
- S1, S2: now not fitted; now left out of the parts list
- U3: value ~ -> SI4909DY-VB
Changed lines of the file:
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@@
   )
   (symbol (lib_id "B3U-1000P:B3U-1000P") (at 33.655 46.355 0) (mirror y) (unit 1)
-    (in_bom yes) (on_board yes) (dnp no) (fields_autoplaced)
+    (in_bom no) (on_board yes) (dnp yes) (fields_autoplaced)
     (property "Reference" "S2" (at 33.655 40.005 0)
       (effects (font (size 1.27 1.27)))
@@
   )
   (symbol (lib_id "Jumper:Jumper_2_Bridged") (at 266.954 100.33 90) (unit 1)
-    (in_bom yes) (on_board yes) (dnp no)
+    (in_bom no) (on_board yes) (dnp no)
     (property "Reference" "JP2" (at 264.414 99.695 90)
       (effects (font (size 1.27 1.27)) (justify left))
@@
   )
   (symbol (lib_id "Jumper:Jumper_2_Bridged") (at 205.74 107.95 270) (mirror x) (unit 1)
-    (in_bom yes) (on_board yes) (dnp no) (fields_autoplaced)
+    (in_bom no) (on_board yes) (dnp no) (fields_autoplaced)
     (property "Reference" "JP1" (at 208.28 107.315 90)
       (effects (font (size 1.27 1.27)) (justify left))
@@
       (effects (font (size 1.27 1.27)))
     )
-    (property "Value" "~" (at 222.25 24.765 0)
+    (property "Value" "SI4909DY-VB" (at 222.25 24.765 0)
       (effects (font (size 1.27 1.27)))
     )
@@
   )
   (symbol (lib_id "RF_Module:ESP32-WROOM-32D") (at 69.85 76.835 0) (unit 1)
-    (in_bom yes) (on_board yes) (dnp no)
+    (in_bom no) (on_board yes) (dnp no)
     (property "Reference" "U5" (at 76.2 124.46 0)
       (effects (font (size 1.27 1.27)) (justify left))
@@
   )
   (symbol (lib_id "B3U-1000P:B3U-1000P") (at 94.615 43.18 0) (mirror y) (unit 1)
-    (in_bom yes) (on_board yes) (dnp no) (fields_autoplaced)
+    (in_bom no) (on_board yes) (dnp yes) (fields_autoplaced)
     (property "Reference" "S1" (at 94.615 37.465 0)
       (effects (font (size 1.27 1.27)))
@@
   )
   (symbol (lib_id "Connector:Screw_Terminal_01x04") (at 168.275 81.28 90) (unit 1)
-    (in_bom no) (on_board yes) (dnp no) (fields_autoplaced)
+    (in_bom no) (on_board yes) (dnp yes) (fields_autoplaced)
     (property "Reference" "J2" (at 169.545 75.565 90)
       (effects (font (size 1.27 1.27)))
