File: kicad/luz/luz.kicad_pcb (KiCad board)
At the start: 4 copper layers, 49.4 x 21.9 mm, 65 parts, among them J2 Screw_Terminal_01x04, Q1 AO3400A, Q4 AO3400A, U1 U261-241N-4BS2SS, U2 CYPD3177-24LQXQ_C2959321, U3 SI4909DY-VB, U4 TPS54302, U5 ESP32-WROOM-32D

Commit message: Typos
Parts:
- moved kibuzzard-655BB485 1.50 mm to (68.3, 115.5), turned to 0 degrees
- moved kibuzzard-655BB458 1.13 mm to (68.7, 99.2), turned to 0 degrees
Changed lines of the file:
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@@
   )
   (footprint "kibuzzard-655BB458" (layer "F.Cu")
-    (at 69.8 99.5 90)
+    (at 68.7 99.25)
     (descr "Generated with KiBuzzard")
     (tags "kb_params=eyJBbGlnbm1lbnRDaG9pY2UiOiAiTGVmdCIsICJDYXBMZWZ0Q2hvaWNlIjogIigiLCAiQ2FwUmlnaHRDaG9pY2UiOiAiKSIsICJGb250Q29tYm9Cb3giOiAiVWJ1bnR1TW9uby1CIiwgIkhlaWdodEN0cmwiOiAiMC44IiwgIkxheWVyQ29tYm9Cb3giOiAiRi5TaWxrUyIsICJNdWx0aUxpbmVUZXh0IjogIkdORCIsICJQYWRkaW5nQm90dG9tQ3RybCI6ICI1IiwgIlBhZGRpbmdMZWZ0Q3RybCI6ICIyIiwgIlBhZGRpbmdSaWdodEN0cmwiOiAiMiIsICJQYWRkaW5nVG9wQ3RybCI6ICI1IiwgIldpZHRoQ3RybCI6ICIifQ==")
     (attr board_only exclude_from_pos_files exclude_from_bom)
-    (fp_text reference "kibuzzard-655BB458" (at 0 -3.722793 90) (layer "F.SilkS") hide
+    (fp_text reference "kibuzzard-655BB458" (at 0 -3.722793) (layer "F.SilkS") hide
         (effects (font (size 0 0) (thickness 0.15)))
     )
-    (fp_text value "G***" (at 0 3.722793 90) (layer "F.SilkS") hide
+    (fp_text value "G***" (at 0 3.722793) (layer "F.SilkS") hide
         (effects (font (size 0 0) (thickness 0.15)))
     )
@@
   )
   (footprint "kibuzzard-655BB485" (layer "F.Cu")
-    (at 69.8 115.5 90)
+    (at 68.3 115.5)
     (descr "Generated with KiBuzzard")
     (tags "kb_params=eyJBbGlnbm1lbnRDaG9pY2UiOiAiTGVmdCIsICJDYXBMZWZ0Q2hvaWNlIjogIigiLCAiQ2FwUmlnaHRDaG9pY2UiOiAiKSIsICJGb250Q29tYm9Cb3giOiAiVWJ1bnR1TW9uby1CIiwgIkhlaWdodEN0cmwiOiAiMC44IiwgIkxheWVyQ29tYm9Cb3giOiAiRi5TaWxrUyIsICJNdWx0aUxpbmVUZXh0IjogIlZPVVQiLCAiUGFkZGluZ0JvdHRvbUN0cmwiOiAiNSIsICJQYWRkaW5nTGVmdEN0cmwiOiAiMiIsICJQYWRkaW5nUmlnaHRDdHJsIjogIjIiLCAiUGFkZGluZ1RvcEN0cmwiOiAiNSIsICJXaWR0aEN0cmwiOiAiIn0=")
     (attr board_only exclude_from_pos_files exclude_from_bom)
-    (fp_text reference "kibuzzard-655BB485" (at 0 -3.722793 90) (layer "F.SilkS") hide
+    (fp_text reference "kibuzzard-655BB485" (at 0 -3.722793) (layer "F.SilkS") hide
         (effects (font (size 0 0) (thickness 0.15)))
     )
-    (fp_text value "G***" (at 0 3.722793 90) (layer "F.SilkS") hide
+    (fp_text value "G***" (at 0 3.722793) (layer "F.SilkS") hide
         (effects (font (size 0 0) (thickness 0.15)))
     )
